File: q1/_saved_qa.sch (KiCad schematic (older format))
At the start: 72 parts, among them IC1 74AHC1G125, J1 Conn_01x02_Female, J2 Barrel_Jack, J3 screw term, J4 Conn_01x01_Female, J5 Connector_Micro_SD_Card, J6 UJ2-MIBH2-4-SMT, J7 Screw_Terminal_01x03, J8 Screw_Terminal_01x06, P1 Conn_01x12_Female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

Commit message: update
Parts:
- J2: footprint (none) -> Connector_BarrelJack:BarrelJack_Horizontal
Changed lines of the file:
@@
 F 0 "J2" H 4405 1225 50  0000 C CNN
 F 1 "Barrel_Jack" H 4405 1134 50  0000 C CNN
-F 2 "" H 4400 860 50  0001 C CNN
+F 2 "Connector_BarrelJack:BarrelJack_Horizontal" H 4400 860 50  0001 C CNN
 F 3 "~" H 4400 860 50  0001 C CNN
 	1    4350 900
