File: q1/_saved_qa.sch (KiCad schematic (older format))
At the start: 79 parts, among them IC1 74AHC1G125, J1 Conn_01x02_Female, J2 Barrel_Jack, J3 Conn_01x02_Female, J4 Conn_01x01_Female, J5 Connector_Micro_SD_Card, J6 UJ2-MIBH2-4-SMT, J8 Screw_Terminal_01x06, P1 Conn_01x12_Female, P2 Conn_01x12_Female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

Commit message: update
Connections:
- net labels added: D8_DONE
- net labels removed: D8, MICRO_DONE_PIN
- wire segments 278 -> 276
Changed lines of the file:
@@
 D9_SD_CS
 Text Label 6100 6000 0    70   ~ 0
-D8
+D8_DONE
 Wire Wire Line
 	5000 7900 5300 7900
@@
 	4250 750  4000 750
 Wire Wire Line
-	1200 1650 1300 1650
-Wire Wire Line
-	1300 1650 1300 2100
-Wire Wire Line
-	1300 2100 1050 2100
-Text GLabel 1050 2100 0    50   Input ~ 0
-MICRO_DONE_PIN
-Wire Wire Line
 	1200 1450 1600 1450
 Wire Wire Line
@@
 	1    0    0    -1
 $EndComp
-Text Notes 3250 450  0    50   ~ 0
+Text Notes 5200 50   0    50   ~ 0
 (VMIN: 6.5V; VMAX: 36V)
 $Comp
@@
 Wire Wire Line
 	3850 3250 3350 3250
-Text Notes 3550 2250 0    50   ~ 0
+Text Notes 5300 1950 0    50   ~ 0
 (VIN MAX: 6V)
 $Comp
@@
 Text Notes 19450 7600 0    59   ~ 0
 TODO: USE THIS FOR M4 XTAL?
-$Comp
-L Connector_Generic:Conn_02x03_Top_Bottom J?
-U 1 1 5D9104F6
-P 2400 1650
-F 0 "J?" H 2450 1967 50  0000 C CNN
-F 1 "Conn_02x03_Top_Bottom" V 2100 1250 50  0000 C CNN
-F 2 "" H 2400 1650 50  0001 C CNN
-F 3 "~" H 2400 1650 50  0001 C CNN
-	1    2400 1650
-	1    0    0    -1
-$EndComp
 Wire Wire Line
 	1200 1550 2200 1550
-Wire Wire Line
-	2200 1550 2200 1650
 Connection ~ 2200 1550
-Wire Wire Line
-	2200 1650 2200 1750
-Connection ~ 2200 1650
 Wire Wire Line
 	3350 1550 3350 3250
@@
 Wire Wire Line
 	1200 300  1200 1250
+Wire Wire Line
+	1200 1650 1550 1650
+Text Label 1250 1650 0    50   ~ 0
+D8_DONE
+Wire Wire Line
+	2200 1650 2200 1750
+Wire Wire Line
+	2200 1550 2200 1650
+Connection ~ 2200 1650
+$Comp
+L Connector_Generic:Conn_02x03_Top_Bottom J?
+U 1 1 5D9104F6
+P 2400 1650
+F 0 "J?" H 2450 1967 50  0000 C CNN
+F 1 "Conn_02x03_Top_Bottom" V 2100 1250 50  0000 C CNN
+F 2 "" H 2400 1650 50  0001 C CNN
+F 3 "~" H 2400 1650 50  0001 C CNN
+	1    2400 1650
+	1    0    0    -1
+$EndComp
 $EndSCHEMATC
