File: q1/qa.kicad_pcb (KiCad board)
At the start: 2 copper layers, 66.4 x 75.6 mm, 62 parts, among them IC1 74AHC1G125, J2 Barrel_Jack, J3 screw term, J5 Connector_Micro_SD_Card, J6 UJ2-MIBH2-4-SMT, J7 Screw_Terminal_01x03, J8 Screw_Terminal_01x06, P1 Conn_01x12_Female, P2 Conn_01x12_Female, U1 tpl5110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

Commit message: update
Parts:
- J3: value screw term -> Conn_01x02_Female; footprint TerminalBlock_Phoenix:TerminalBlock_Phoenix_PT-1,5-2-3.5-H_1x02_P3.50mm_Horizontal -> Connector_JST:JST_PH_S2B-PH-SM4-TB_1x02-1MP_P2.00mm_Horizontal
- moved X1 3.85 mm to (57.2, 88.4)
- moved J3 0.46 mm to (69.3, 87.7)
Connections:
- J3 pad 1: (no net) -> GND
- J3 pad 2: GND -> (no net)
Changed lines of the file:
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@@
   )
   (module qa:4UCONN_20329_V2 (layer F.Cu)
-    (at 61.0235 88.8873)
+    (at 57.2008 88.4174)
     (fp_text reference X1 (at -2.778 5.852 -180) (layer F.SilkS)
       (effects (font (size 0.9652 0.9652) (thickness 0.173736)) (justify right top))
@@
     (pad 1 thru_hole circle (at 0 0) (size 4.5 4.5) (drill 2.7) (layers *.Cu *.Mask))
   )
-  (module TerminalBlock_Phoenix:TerminalBlock_Phoenix_PT-1,5-2-3.5-H_1x02_P3.50mm_Horizontal (layer F.Cu)
-    (at 69.5579 87.9983)
-    (descr "Terminal Block Phoenix PT-1,5-2-3.5-H, 2 pins, pitch 3.5mm, size 7x7.6mm^2, drill diamater 1.2mm, pad diameter 2.4mm, see , script-generated using https://github.com/pointhi/kicad-footprint-generator/scripts/TerminalBlock_Phoenix")
-    (tags "THT Terminal Block Phoenix PT-1,5-2-3.5-H pitch 3.5mm size 7x7.6mm^2 drill 1.2mm pad 2.4mm")
-    (fp_text reference J3 (at 1.75 -4.16) (layer F.SilkS)
-      (effects (font (size 1 1) (thickness 0.15)))
-    )
-    (fp_text value "screw term" (at 1.75 5.56) (layer F.Fab)
-      (effects (font (size 1 1) (thickness 0.15)))
-    )
-    (fp_arc (start 0 0) (end 0 1.68) (angle -32) (layer F.SilkS) (width 0.12))
-    (fp_arc (start 0 0) (end 1.425 0.891) (angle -64) (layer F.SilkS) (width 0.12))
-    (fp_arc (start 0 0) (end 0.866 -1.44) (angle -63) (layer F.SilkS) (width 0.12))
-    (fp_arc (start 0 0) (end -1.44 -0.866) (angle -63) (layer F.SilkS) (width 0.12))
-    (fp_arc (start 0 0) (end -0.866 1.44) (angle -32) (layer F.SilkS) (width 0.12))
-    (fp_circle (center 0 0) (end 1.5 0) (layer F.Fab) (width 0.1))
-    (fp_circle (center 3.5 0) (end 5 0) (layer F.Fab) (width 0.1))
-    (fp_circle (center 3.5 0) (end 5.18 0) (layer F.SilkS) (width 0.12))
-    (fp_line (start -1.75 -3.1) (end 5.25 -3.1) (layer F.Fab) (width 0.1))
-    (fp_line (start 5.25 -3.1) (end 5.25 4.5) (layer F.Fab) (width 0.1))
-    (fp_line (start 5.25 4.5) (end -1.35 4.5) (layer F.Fab) (width 0.1))
-    (fp_line (start -1.35 4.5) (end -1.75 4.1) (layer F.Fab) (width 0.1))
-    (fp_line (start -1.75 4.1) (end -1.75 -3.1) (layer F.Fab) (width 0.1))
-    (fp_line (start -1.75 4.1) (end 5.25 4.1) (layer F.Fab) (width 0.1))
-    (fp_line (start -1.81 4.1) (end 5.31 4.1) (layer F.SilkS) (width 0.12))
-    (fp_line (start -1.75 3) (end 5.25 3) (layer F.Fab) (width 0.1))
-    (fp_line (start -1.81 3) (end 5.31 3) (layer F.SilkS) (width 0.12))
-    (fp_line (start -1.81 -3.16) (end 5.31 -3.16) (layer F.SilkS) (width 0.12))
-    (fp_line (start -1.81 4.56) (end 5.31 4.56) (layer F.SilkS) (width 0.12))
-    (fp_line (start -1.81 -3.16) (end -1.81 4.56) (layer F.SilkS) (width 0.12))
-    (fp_line (start 5.31 -3.16) (end 5.31 4.56) (layer F.SilkS) (width 0.12))
-    (fp_line (start 1.138 -0.955) (end -0.955 1.138) (layer F.Fab) (width 0.1))
-    (fp_line (start 0.955 -1.138) (end -1.138 0.955) (layer F.Fab) (width 0.1))
-    (fp_line (start 4.638 -0.955) (end 2.546 1.138) (layer F.Fab) (width 0.1))
-    (fp_line (start 4.455 -1.138) (end 2.363 0.955) (layer F.Fab) (width 0.1))
-    (fp_line (start 4.775 -1.069) (end 4.646 -0.941) (layer F.SilkS) (width 0.12))
-    (fp_line (start 2.525 1.181) (end 2.431 1.274) (layer F.SilkS) (width 0.12))
-    (fp_line (start 4.57 -1.275) (end 4.476 -1.181) (layer F.SilkS) (width 0.12))
-    (fp_line (start 2.355 0.941) (end 2.226 1.069) (layer F.SilkS) (width 0.12))
-    (fp_line (start -2.05 4.16) (end -2.05 4.8) (layer F.SilkS) (width 0.12))
-    (fp_line (start -2.05 4.8) (end -1.65 4.8) (layer F.SilkS) (width 0.12))
-    (fp_line (start -2.25 -3.6) (end -2.25 5) (layer F.CrtYd) (width 0.05))
-    (fp_line (start -2.25 5) (end 5.75 5) (layer F.CrtYd) (width 0.05))
-    (fp_line (start 5.75 5) (end 5.75 -3.6) (layer F.CrtYd) (width 0.05))
-    (fp_line (start 5.75 -3.6) (end -2.25 -3.6) (layer F.CrtYd) (width 0.05))
-    (fp_text user %R (at 1.75 2.4) (layer F.Fab)
-      (effects (font (size 1 1) (thickness 0.15)))
-    )
-    (pad 1 thru_hole rect (at 0 0) (size 2.4 2.4) (drill 1.2) (layers *.Cu *.Mask))
-    (pad 2 thru_hole circle (at 3.5 0) (size 2.4 2.4) (drill 1.2) (layers *.Cu *.Mask)
-      (net 8 GND))
-    (model ${KISYS3DMOD}/TerminalBlock_Phoenix.3dshapes/TerminalBlock_Phoenix_PT-1,5-2-3.5-H_1x02_P3.50mm_Horizontal.wrl
-      (at (xyz 0 0 0))
-      (scale (xyz 1 1 1))
-      (rotate (xyz 0 0 0))
-    )
-  )
   (module TerminalBlock_Phoenix:TerminalBlock_Phoenix_PT-1,5-3-3.5-H_1x03_P3.50mm_Horizontal (layer F.Cu)
     (at 104.3559 74.0791 90)
@@
       (at (xyz 0 0 0))
       (scale (xyz 1 1 1))
+      (rotate (xyz 0 0 0))
+    )
+  )
+  (module Connector_JST:JST_PH_S2B-PH-SM4-TB_1x02-1MP_P2.00mm_Horizontal (layer F.Cu)
+    (at 69.2531 87.6554)
+    (descr "JST PH series connector, S2B-PH-SM4-TB (http://www.jst-mfg.com/product/pdf/eng/ePH.pdf), generated with kicad-footprint-generator")
+    (tags "connector JST PH top entry")
+    (attr smd)
+    (fp_text reference J3 (at 0 -5.8) (layer F.SilkS)
+      (effects (font (size 1 1) (thickness 0.15)))
+    )
+    (fp_text value Conn_01x02_Female (at 0 5.8) (layer F.Fab)
+      (effects (font (size 1 1) (thickness 0.15)))
+    )
+    (fp_line (start -3.95 -3.2) (end -3.15 -3.2) (layer F.Fab) (width 0.1))
+    (fp_line (start -3.15 -3.2) (end -3.15 -1.6) (layer F.Fab) (width 0.1))
+    (fp_line (start -3.15 -1.6) (end 3.15 -1.6) (layer F.Fab) (width 0.1))
+    (fp_line (start 3.15 -1.6) (end 3.15 -3.2) (layer F.Fab) (width 0.1))
+    (fp_line (start 3.15 -3.2) (end 3.95 -3.2) (layer F.Fab) (width 0.1))
+    (fp_line (start -4.06 0.94) (end -4.06 -3.31) (layer F.SilkS) (width 0.12))
+    (fp_line (start -4.06 -3.31) (end -3.04 -3.31) (layer F.SilkS) (width 0.12))
+    (fp_line (start -3.04 -3.31) (end -3.04 -1.71) (layer F.SilkS) (width 0.12))
+    (fp_line (start -3.04 -1.71) (end -1.76 -1.71) (layer F.SilkS) (width 0.12))
+    (fp_line (start -1.76 -1.71) (end -1.76 -4.6) (layer F.SilkS) (width 0.12))
+    (fp_line (start 4.06 0.94) (end 4.06 -3.31) (layer F.SilkS) (width 0.12))
+    (fp_line (start 4.06 -3.31) (end 3.04 -3.31) (layer F.SilkS) (width 0.12))
+    (fp_line (start 3.04 -3.31) (end 3.04 -1.71) (layer F.SilkS) (width 0.12))
+    (fp_line (start 3.04 -1.71) (end 1.76 -1.71) (layer F.SilkS) (width 0.12))
+    (fp_line (start -2.34 4.51) (end 2.34 4.51) (layer F.SilkS) (width 0.12))
+    (fp_line (start -3.95 4.4) (end 3.95 4.4) (layer F.Fab) (width 0.1))
+    (fp_line (start -3.95 -3.2) (end -3.95 4.4) (layer F.Fab) (width 0.1))
+    (fp_line (start 3.95 -3.2) (end 3.95 4.4) (layer F.Fab) (width 0.1))
+    (fp_line (start -4.6 -5.1) (end -4.6 5.1) (layer F.CrtYd) (width 0.05))
+    (fp_line (start -4.6 5.1) (end 4.6 5.1) (layer F.CrtYd) (width 0.05))
+    (fp_line (start 4.6 5.1) (end 4.6 -5.1) (layer F.CrtYd) (width 0.05))
+    (fp_line (start 4.6 -5.1) (end -4.6 -5.1) (layer F.CrtYd) (width 0.05))
+    (fp_line (start -1.5 -1.6) (end -1 -0.892893) (layer F.Fab) (width 0.1))
+    (fp_line (start -1 -0.892893) (end -0.5 -1.6) (layer F.Fab) (width 0.1))
+    (fp_text user %R (at 0 1.5) (layer F.Fab)
+      (effects (font (size 1 1) (thickness 0.15)))
+    )
+    (pad 1 smd roundrect (at -1 -2.85) (size 1 3.5) (layers F.Cu F.Paste F.Mask) (roundrect_rratio 0.25)
+      (net 8 GND))
+    (pad 2 smd roundrect (at 1 -2.85) (size 1 3.5) (layers F.Cu F.Paste F.Mask) (roundrect_rratio 0.25))
+    (pad MP smd roundrect (at -3.35 2.9) (size 1.5 3.4) (layers F.Cu F.Paste F.Mask) (roundrect_rratio 0.166667))
+    (pad MP smd roundrect (at 3.35 2.9) (size 1.5 3.4) (layers F.Cu F.Paste F.Mask) (roundrect_rratio 0.166667))
+    (model ${KISYS3DMOD}/Connector_JST.3dshapes/JST_PH_S2B-PH-SM4-TB_1x02-1MP_P2.00mm_Horizontal.wrl
+      (at (xyz 0 0 0))
+      (scale (xyz 1 1 1))

Commit message: update
Parts:
- removed J7: Screw_Terminal_01x03, TerminalBlock_Phoenix:TerminalBlock_Phoenix_PT-1,5-3-3.5-H_1x03_P3.50mm_Horizontal
- added BT1: Battery_Cell, Battery:BatteryHolder_Keystone_3000_1x12mm, F.Cu at (121.1, 59.7)
- added OWS1: Screw_Terminal_01x03, TerminalBlock_Phoenix:TerminalBlock_Phoenix_PT-1,5-3-3.5-H_1x03_P3.50mm_Horizontal, F.Cu at (144.4, 22.9)
- U$1: footprint qa:PQFN64-1 -> Package_QFP:TQFP-64-1EP_10x10mm_P0.5mm_EP8x8mm
- moved R10 30.2 mm to (117.7, 103.6)
- moved R12 25.0 mm to (112.8, 112.0)
- moved R11 15.6 mm to (125.0, 118.3)
Connections:
- U1 pad 1: (no net) -> Net-(BT1-Pad1)
