File: q1/qa.sch (KiCad schematic (older format))
At the start: 72 parts, among them IC1 74AHC1G125, J1 Conn_01x02_Female, J2 Barrel_Jack, J3 screw term, J4 Conn_01x01_Female, J5 Connector_Micro_SD_Card, J6 UJ2-MIBH2-4-SMT, J7 Screw_Terminal_01x03, J8 Screw_Terminal_01x06, P1 Conn_01x12_Female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

Commit message: update
Parts:
- removed J3: screw term, TerminalBlock_Phoenix:TerminalBlock_Phoenix_PT-1,5-2-3.5-H_1x02_P3.50mm_Horizontal, symbol Connector:Screw_Terminal_01x02
- added J3: Conn_01x02_Female, Connector_JST:JST_PH_S2B-PH-SM4-TB_1x02-1MP_P2.00mm_Horizontal, symbol Connector:Conn_01x02_Female
- J2: footprint (none) -> Connector_BarrelJack:BarrelJack_Horizontal
Other:
- moved on the sheet: J7, J8
Changed lines of the file:
@@
 	4900 2500 4650 2500
-$Comp
-L Connector:Screw_Terminal_01x02 J3
-U 1 1 5DB1B2FB
-P 4450 2500
-F 0 "J3" H 4450 2250 50  0000 C CNN
-F 1 "screw term" V 4600 2450 50  0000 C CNN
-F 2 "TerminalBlock_Phoenix:TerminalBlock_Phoenix_PT-1,5-2-3.5-H_1x02_P3.50mm_Horizontal" H 4450 2500 50  0001 C CNN
-F 3 "~" H 4450 2500 50  0001 C CNN
-	1    4450 2500
-	-1   0    0    -1
-$EndComp
 $Comp
 L power:GND #PWR0112
@@
 F 0 "J2" H 4405 1225 50  0000 C CNN
 F 1 "Barrel_Jack" H 4405 1134 50  0000 C CNN
-F 2 "" H 4400 860 50  0001 C CNN
+F 2 "Connector_BarrelJack:BarrelJack_Horizontal" H 4400 860 50  0001 C CNN
 F 3 "~" H 4400 860 50  0001 C CNN
 	1    4350 900
@@
 L Connector:Screw_Terminal_01x03 J7
 U 1 1 5DC30348
-P -550 3850
-F 0 "J7" H -470 3892 50  0000 L CNN
-F 1 "Screw_Terminal_01x03" H -470 3801 50  0000 L CNN
-F 2 "TerminalBlock_Phoenix:TerminalBlock_Phoenix_PT-1,5-3-3.5-H_1x03_P3.50mm_Horizontal" H -550 3850 50  0001 C CNN
-F 3 "~" H -550 3850 50  0001 C CNN
-	1    -550 3850
+P 10600 3100
+F 0 "J7" H 10680 3142 50  0000 L CNN
+F 1 "Screw_Terminal_01x03" H 10680 3051 50  0000 L CNN
+F 2 "TerminalBlock_Phoenix:TerminalBlock_Phoenix_PT-1,5-3-3.5-H_1x03_P3.50mm_Horizontal" H 10600 3100 50  0001 C CNN
+F 3 "~" H 10600 3100 50  0001 C CNN
+	1    10600 3100
 	1    0    0    -1
 $EndComp
@@
 L Connector:Screw_Terminal_01x06 J8
 U 1 1 5DC3086D
-P -550 5000
-F 0 "J8" H -470 4992 50  0000 L CNN
-F 1 "Screw_Terminal_01x06" H -470 4901 50  0000 L CNN
-F 2 "TerminalBlock_Phoenix:TerminalBlock_Phoenix_PT-1,5-6-3.5-H_1x06_P3.50mm_Horizontal" H -550 5000 50  0001 C CNN
-F 3 "~" H -550 5000 50  0001 C CNN
-	1    -550 5000
-	1    0    0    -1
+P 10600 4250
+F 0 "J8" H 10680 4242 50  0000 L CNN
+F 1 "Screw_Terminal_01x06" H 10680 4151 50  0000 L CNN
+F 2 "TerminalBlock_Phoenix:TerminalBlock_Phoenix_PT-1,5-6-3.5-H_1x06_P3.50mm_Horizontal" H 10600 4250 50  0001 C CNN
+F 3 "~" H 10600 4250 50  0001 C CNN
+	1    10600 4250
+	1    0    0    -1
+$EndComp
+$Comp
+L Connector:Conn_01x02_Female J3
+U 1 1 5DC5D8BB
+P 4450 2600
+F 0 "J3" H 4344 2275 50  0000 C CNN
+F 1 "Conn_01x02_Female" H 4344 2366 50  0000 C CNN
+F 2 "Connector_JST:JST_PH_S2B-PH-SM4-TB_1x02-1MP_P2.00mm_Horizontal" H 4450 2600 50  0001 C CNN
+F 3 "~" H 4450 2600 50  0001 C CNN
+	1    4450 2600
+	-1   0    0    1
 $EndComp
 $EndSCHEMATC

Commit message: update
Parts:
- removed J7: Screw_Terminal_01x03, TerminalBlock_Phoenix:TerminalBlock_Phoenix_PT-1,5-3-3.5-H_1x03_P3.50mm_Horizontal, symbol Connector:Screw_Terminal_01x03
- added J?: Conn_02x03_Top_Bottom, symbol Connector_Generic:Conn_02x03_Top_Bottom
- added J?: Conn_01x01_Female, symbol Connector:Conn_01x01_Female
- added JP?: Jumper_2_Bridged, symbol Jumper:Jumper_2_Bridged
- added OWS1: Screw_Terminal_01x03, TerminalBlock_Phoenix:TerminalBlock_Phoenix_PT-1,5-3-3.5-H_1x03_P3.50mm_Horizontal, symbol Connector:Screw_Terminal_01x03
- added SW? (x2): SW_DPDT_x2, symbol Switch:SW_DPDT_x2
- added SW?: SWITCH_SPDT, symbol qa-eagle-import:SWITCH_SPDT
- added U?: DS3231MZ, Package_SO:SOIC-8_3.9x4.9mm_P1.27mm, symbol Timer_RTC:DS3231MZ
- BT1: footprint (none) -> Battery:BatteryHolder_Keystone_3000_1x12mm
- U$1: footprint qa:PQFN64-1 -> Package_QFP:TQFP-64-1EP_10x10mm_P0.5mm_EP8x8mm
Connections:
- net labels added: D5_LORA_CS, D5_LORA_RESET, D7_LORA_CS, D7_LORA_RESET, D8_DONE, D9_SD_CS, RTC_32KHZ, RTC_~INT, RTC_~RST
- net labels removed: D5, D7, D8, LORA_CS, LORA_RESET, MICRO_DONE_PIN, SD_CS
- wire segments 255 -> 276
Other:
- note added: "ADDITIONAL UARTS:\n D2, A4\n A3, A2\n A1, A5"
- note added: "Crypto"
- note added: "External Serial"
- note added: "I2C Pullups"
- note added: "One-Wire"
- note added: "RTC DS3231"
- note added: "TODO: USE THIS FOR M4 XTAL?"
- moved on the sheet: BT1, D1, D2, D3, J1, J2, J3, J6, J8, Q1, Q2, Q3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

Commit message: update
Parts:
- added C? (x7): C, symbol Device:C
- added L?: L, symbol Device:L
- added R? (x4): R, symbol Device:R
- added U?: LTC3114-1, symbol qa_dwb:LTC3114-1
Connections:
- net labels added: VIN, VOUT
- wire segments 276 -> 330
