File: q3/ib4/ib4/ib4.kicad_pcb (KiCad board)
At the start: 4 copper layers, 102.6 x 67.8 mm, 11 parts, among them J1 Conn_01x12_Female, J2 Conn_01x09_Female, J3 Screw_Terminal_01x02, J4 Conn_01x08_Female

Commit message: update
Connections:
- J1 pad 7: E_~RST -> E_CS
- J1 pad 8: E_CS -> E_BUSY
- J1 pad 9: E_BUSY -> E_~RST
- JP2 pad 5: E_~RST -> E_CS
- JP2 pad 6: E_CS -> E_BUSY
- JP2 pad 7: E_BUSY -> E_~RST
